File: khonsu.kicad_pcb (KiCad board)
At the start: 2 copper layers, 232 x 90 mm, 85 parts

Commit message: Add khonsu file
Parts:
- removed the ? at (134.0, 70.0)
- removed D2:2 (x42): , DIODE
- removed SW0:0, SW0:1, SW0:2, SW0:3, SW10:0, SW10:1, SW10:2, SW10:3, SW11:0, SW11:1, SW11:2, SW11:3, SW1:0, SW1:1, SW1:2, SW1:3, SW2:0, SW2:1, SW2:2, SW2:3, SW3:0, SW3:1, SW3:2, SW3:3, SW4:0, SW4:1, SW4:2, SW4:3, SW5:0, SW6:0, SW7:0, SW7:1, SW7:2, SW7:3, SW8:0, SW8:1, SW8:2, SW8:3, SW9:0, SW9:1, SW9:2, SW9:3: , MX_FLIP
- added ?: , pcb-element-thru-holes,  at (109.5, 74.5)
- added D**: D, khonsu-diode-front, F.Cu at (151.0, 72.0)
- added D**: D, khonsu-diode-front, F.Cu at (141.0, 84.0)
- added D**: D, khonsu-diode-front, F.Cu at (141.0, 96.0)
- added D**: D, khonsu-diode-front, F.Cu at (136.0, 72.0)
- added D**: D, khonsu-diode-front, F.Cu at (136.0, 84.0)
- added D**: D, khonsu-diode-front, F.Cu at (136.0, 96.0)
- added D**: D, khonsu-diode-front, F.Cu at (131.0, 72.0)
- added D**: D, khonsu-diode-front, F.Cu at (131.0, 84.0)
- added D**: D, khonsu-diode-front, F.Cu at (131.0, 96.0)
- added D**: D, khonsu-diode-front, F.Cu at (156.0, 72.0)
- added D**: D, khonsu-diode-back, B.Cu at (156.0, 84.0)
- added D**: D, khonsu-diode-front, F.Cu at (151.0, 84.0)
- added D**: D, khonsu-diode-back, B.Cu at (161.0, 72.0)
- added D**: D, khonsu-diode-back, B.Cu at (161.0, 84.0)
- added D**: D, khonsu-diode-back, B.Cu at (161.0, 96.0)
- added D**: D, khonsu-diode-back, B.Cu at (161.0, 108.0)
- added D**: D, khonsu-diode-back, B.Cu at (166.0, 72.0)
- added D**: D, khonsu-diode-back, B.Cu at (166.0, 84.0)
- added D**: D, khonsu-diode-back, B.Cu at (166.0, 96.0)
- added D**: D, khonsu-diode-back, B.Cu at (166.0, 108.0)
- added D**: D, khonsu-diode-back, B.Cu at (171.0, 72.0)
- added D**: D, khonsu-diode-back, B.Cu at (171.0, 84.0)
- added D**: D, khonsu-diode-front, F.Cu at (151.0, 96.0)
- added D**: D, khonsu-diode-back, B.Cu at (171.0, 96.0)
- added D**: D, khonsu-diode-back, B.Cu at (176.0, 72.0)
- added D**: D, khonsu-diode-back, B.Cu at (176.0, 84.0)
- added D**: D, khonsu-diode-back, B.Cu at (176.0, 96.0)
- added D**: D, khonsu-diode-back, B.Cu at (181.0, 72.0)
- added D**: D, khonsu-diode-back, B.Cu at (181.0, 84.0)
- added D**: D, khonsu-diode-back, B.Cu at (181.0, 96.0)
- added D**: D, khonsu-diode-front, F.Cu at (151.0, 108.0)
- added D**: D, khonsu-diode-front, F.Cu at (146.0, 72.0)
- added D**: D, khonsu-diode-front, F.Cu at (146.0, 84.0)
- added D**: D, khonsu-diode-front, F.Cu at (146.0, 96.0)
- added D**: D, khonsu-diode-front, F.Cu at (146.0, 108.0)
- added D**: D, khonsu-diode-front, F.Cu at (141.0, 72.0)
- added REF**: Kailh_socket_MX_optional_reversible, Kailh_socket_MX_optional_reversible_platemount, F.Cu at (112.7, 41.6)
- added REF**: Kailh_socket_MX_optional_reversible, Kailh_socket_MX_optional_reversible_platemount, F.Cu at (65.3, 41.8)
- added REF**: Kailh_socket_MX_optional_reversible, Kailh_socket_MX_optional_reversible_platemount, F.Cu at (60.4, 60.1)
- added REF**: Kailh_socket_MX_optional_reversible, Kailh_socket_MX_optional_reversible_platemount, F.Cu at (51.3, 20.8)
- added REF**: Kailh_socket_MX_optional_reversible, Kailh_socket_MX_optional_reversible_platemount, F.Cu at (46.4, 39.2)
- added REF**: Kailh_socket_MX_optional_reversible, Kailh_socket_MX_optional_reversible_platemount, F.Cu at (41.4, 57.5)
- added REF**: Kailh_socket_MX_optional_reversible, Kailh_socket_MX_optional_reversible_platemount, F.Cu at (24.4, 26.8)
- added REF**: Kailh_socket_MX_optional_reversible, Kailh_socket_MX_optional_reversible_platemount, F.Cu at (22.3, 45.7)
- added REF**: Kailh_socket_MX_optional_reversible, Kailh_socket_MX_optional_reversible_platemount, F.Cu at (20.3, 64.5)
- added REF**: Kailh_socket_MX_optional_reversible, Kailh_socket_MX_optional_reversible_platemount, F.Cu at (102.5, 110.9)
- added REF**: Kailh_socket_MX_optional_reversible, Kailh_socket_MX_optional_reversible_platemount, F.Cu at (201.7, 110.9)
- added REF**: Kailh_socket_MX_optional_reversible, Kailh_socket_MX_optional_reversible_platemount, F.Cu at (104.7, 58.8)
- added REF**: Kailh_socket_MX_optional_reversible, Kailh_socket_MX_optional_reversible_platemount, F.Cu at (191.5, 41.6)
- added REF**: Kailh_socket_MX_optional_reversible, Kailh_socket_MX_optional_reversible_platemount, F.Cu at (199.6, 58.8)
- added REF**: Kailh_socket_MX_optional_reversible, Kailh_socket_MX_optional_reversible_platemount, F.Cu at (207.6, 76.1)
- added REF**: Kailh_socket_MX_optional_reversible, Kailh_socket_MX_optional_reversible_platemount, F.Cu at (216.2, 94.8)
- added REF**: Kailh_socket_MX_optional_reversible, Kailh_socket_MX_optional_reversible_platemount, F.Cu at (212.5, 31.8)
- added REF**: Kailh_socket_MX_optional_reversible, Kailh_socket_MX_optional_reversible_platemount, F.Cu at (219.0, 49.7)
- added REF**: Kailh_socket_MX_optional_reversible, Kailh_socket_MX_optional_reversible_platemount, F.Cu at (225.5, 67.5)
- added REF**: Kailh_socket_MX_optional_reversible, Kailh_socket_MX_optional_reversible_platemount, F.Cu at (235.4, 84.1)
- added REF**: Kailh_socket_MX_optional_reversible, Kailh_socket_MX_optional_reversible_platemount, F.Cu at (234.0, 23.4)
- added REF**: Kailh_socket_MX_optional_reversible, Kailh_socket_MX_optional_reversible_platemount, F.Cu at (238.9, 41.8)
- added REF**: Kailh_socket_MX_optional_reversible, Kailh_socket_MX_optional_reversible_platemount, F.Cu at (96.6, 76.1)
- added REF**: Kailh_socket_MX_optional_reversible, Kailh_socket_MX_optional_reversible_platemount, F.Cu at (243.8, 60.1)
- added REF**: Kailh_socket_MX_optional_reversible, Kailh_socket_MX_optional_reversible_platemount, F.Cu at (253.0, 20.8)
- added REF**: Kailh_socket_MX_optional_reversible, Kailh_socket_MX_optional_reversible_platemount, F.Cu at (257.9, 39.2)
- added REF**: Kailh_socket_MX_optional_reversible, Kailh_socket_MX_optional_reversible_platemount, F.Cu at (262.8, 57.5)
- added REF**: Kailh_socket_MX_optional_reversible, Kailh_socket_MX_optional_reversible_platemount, F.Cu at (279.8, 26.8)
- added REF**: Kailh_socket_MX_optional_reversible, Kailh_socket_MX_optional_reversible_platemount, F.Cu at (281.9, 45.7)
- added REF**: Kailh_socket_MX_optional_reversible, Kailh_socket_MX_optional_reversible_platemount, F.Cu at (283.9, 64.5)
- added REF**: Kailh_socket_MX_optional_reversible, Kailh_socket_MX_optional_reversible_platemount, F.Cu at (88.0, 94.8)
- added REF**: Kailh_socket_MX_optional_reversible, Kailh_socket_MX_optional_reversible_platemount, F.Cu at (91.7, 31.8)
- added REF**: Kailh_socket_MX_optional_reversible, Kailh_socket_MX_optional_reversible_platemount, F.Cu at (85.2, 49.7)
- added REF**: Kailh_socket_MX_optional_reversible, Kailh_socket_MX_optional_reversible_platemount, F.Cu at (78.7, 67.5)
- added REF**: Kailh_socket_MX_optional_reversible, Kailh_socket_MX_optional_reversible_platemount, F.Cu at (68.9, 84.1)
- added REF**: Kailh_socket_MX_optional_reversible, Kailh_socket_MX_optional_reversible_platemount, F.Cu at (70.2, 23.4)
- added U1: ProMicro, ArduinoProMicro, F.Cu at (150.0, 35.5)
Routing:
- net N-row-3: track 299.5 -> 0.00 mm
- net N-row-2: track 281.8 -> 0.00 mm
- net N-row-0: track 264.8 -> 0.00 mm
- net N-row-1: track 226.9 -> 0.00 mm
- net N-col-0: track 218.7 -> 0.00 mm, vias 1 -> 0
- net N-col-10: track 211.5 -> 0.00 mm, vias 1 -> 0
- net N-col-1: track 197.0 -> 0.00 mm, vias 1 -> 0
- net N-col-9: track 193.0 -> 0.00 mm, vias 1 -> 0
- net N-col-2: track 189.2 -> 0.00 mm
- net N-col-8: track 176.2 -> 0.00 mm
- net N-col-3: track 162.6 -> 0.00 mm
- net N-col-7: track 153.6 -> 0.00 mm
- net N-col-6: track 124.5 -> 0.00 mm
- net N-col-4: track 124.1 -> 0.00 mm
- net N-col-5: track 80.4 -> 0.00 mm
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Other:
- board size 232 x 90 mm -> 300 x 150 mm
